File: hw/sch_pcb/GPS02A.kicad_pcb (KiCad board)
At the start: 2 copper layers, 60.5 x 40.1 mm, 63 parts, among them J1 HEADER_2x03_PARALLEL, J10 HEADER_2x01_PARALLEL, J11 HEADER_2x01_PARALLEL, J12 HEADER_2x01_PARALLEL, J13 HEADER_2x01_PARALLEL, J14 HEADER_2x01_PARALLEL, J15 HEADER_2x03_PARALLEL, J16 HEADER_2x01_PARALLEL, J17 u.FL, J18 SMA, J2 USB_B, J3 HEADER_2x03_PARALLEL, J4 HEADER_2x01_PARALLEL, J5 HEADER_2x01_PARALLEL, J6 HEADER_2x01_PARALLEL, J7 HEADER_2x01_PARALLEL, J8 HEADER_2x01_PARALLEL, J9 HEADER_2x01_PARALLEL, M1 HOLE, M2 HOLE, M3 HOLE, M4 HOLE, U1 USBLC6-2SC6, U2 MIC5504-3.3YM5, U3 NEO-M8P

Commit message: Update PCB component parameters from schematics.
Connections:
- U2 pad 4: Net-(U2-Pad4) -> unconnected-(U2-Pad4)
- U3 pad 17: Net-(U3-Pad17) -> unconnected-(U3-Pad17)
Other:
- net class Default removed
- net class MLAB_power removed
