File: hw/sch_pcb/GPS02B.kicad_pcb (KiCad board)
At the start: 2 copper layers, 60.5 x 40.1 mm, 64 parts, among them J1 HEADER_2x03_PARALLEL, J10 HEADER_2x01_PARALLEL, J11 HEADER_2x01_PARALLEL, J12 HEADER_2x01_PARALLEL, J13 HEADER_2x01_PARALLEL, J14 HEADER_2x01_PARALLEL, J15 HEADER_2x03_PARALLEL, J16 HEADER_2x01_PARALLEL, J18 SMA, J2 USB_B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

Commit message: Edit bom
Changed lines of the file:
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@@
-(kicad_pcb (version 20210228) (generator pcbnew)
+(kicad_pcb (version 20211014) (generator pcbnew)
   (general
     (thickness 1.6)
@@
     (property "Sheetfile" "GPS02B.kicad_sch")
     (property "Sheetname" "")
-    (property "UST_ID" "")
+    (property "UST_ID" "5c70984712875079b91f8b38")
     (attr smd)
     (fp_text reference "C7" (at 0 0.3175) (layer "B.Fab")
@@
       (effects (font (size 1 1) (thickness 0.15)) (justify mirror))
     )
-    (fp_text value "M4" (at 0 -2.6 180) (layer "B.Fab")
+    (fp_text value "M4" (at 0 -2.6 180) (layer "B.Fab") hide
       (effects (font (size 1 1) (thickness 0.15)) (justify mirror))
     )
-    (fp_text user "${REFERENCE}" (at 0 2.5 180) (layer "B.Fab")
+    (fp_text user "${REFERENCE}" (at -0.191 -2.561 180) (layer "B.Fab")
       (effects (font (size 1 1) (thickness 0.15)) (justify mirror))
     )
@@
     (fp_line (start 0.50118 -0.00102) (end 1.4994 -0.00102) (layer "B.Fab") (width 0.1))
     (pad "1" smd rect locked (at -2 0) (size 2.5 1.8) (layers "B.Cu" "B.Paste" "B.Mask")
-      (net 2 "/VBACKUP") (pinfunction "K"))
+      (net 2 "/VBACKUP") (pinfunction "K") (pintype "passive"))
     (pad "2" smd rect locked (at 2 0) (size 2.5 1.8) (layers "B.Cu" "B.Paste" "B.Mask")
-      (net 6 "Net-(D1-Pad2)") (pinfunction "A"))
+      (net 6 "Net-(D1-Pad2)") (pinfunction "A") (pintype "passive"))
     (model "${KISYS3DMOD}/Diode_SMD.3dshapes/D_SMA.wrl"
       (offset (xyz 0 0 0))
@@
       (effects (font (size 1 1) (thickness 0.15)) (justify mirror))
     )
-    (fp_text value "M4" (at 0 -2.6 90) (layer "B.Fab")
+    (fp_text value "M4" (at 0 -2.6 90) (layer "B.Fab") hide
       (effects (font (size 1 1) (thickness 0.15)) (justify mirror))
     )
-    (fp_text user "${REFERENCE}" (at 0 2.5 90) (layer "B.Fab")
+    (fp_text user "${REFERENCE}" (at -3.048 0 180) (layer "B.Fab")
       (effects (font (size 1 1) (thickness 0.15)) (justify mirror))
     )
@@
     (property "Sheetfile" "GPS02B.kicad_sch")
     (property "Sheetname" "")
-    (property "UST_ID" "")
+    (property "UST_ID" "618cbf071287506e2801ed7e")
     (attr smd)
     (fp_text reference "L2" (at 0 1.17 90) (layer "B.SilkS")
       (effects (font (size 1 1) (thickness 0.15)) (justify mirror))
     )
-    (fp_text value "27nH" (at 0 -1.17 90) (layer "B.Fab")
+    (fp_text value "27nH" (at 0 -1.17 90) (layer "B.Fab") hide
       (effects (font (size 1 1) (thickness 0.15)) (justify mirror))
     )
@@
     (fp_line (start -6.1 8) (end -6.1 -8) (layer "B.Fab") (width 0.1))
     (pad "1" smd rect locked (at -6 7 270) (size 1.8 0.8) (layers "B.Cu" "B.Paste" "B.Mask")
-      (net 42 "/#SAFEB") (pinfunction "~SAFEBOOT") (pintype "input"))
+      (net 42 "/#SAFEB") (pinfunction "~{SAFEBOOT}") (pintype "input"))
     (pad "2" smd rect locked (at -6 5.9 270) (size 1.8 0.8) (layers "B.Cu" "B.Paste" "B.Mask")
       (net 45 "/D_SEL") (pinfunction "D_SEL") (pintype "input"))
@@
       (net 44 "/VDD_USB") (pinfunction "VDD_USB") (pintype "power_in"))
     (pad "8" smd rect locked (at -6 -2.6 270) (size 1.8 0.8) (layers "B.Cu" "B.Paste" "B.Mask")
-      (net 43 "/#RESET") (pinfunction "~RESET") (pintype "input"))
+      (net 43 "/#RESET") (pinfunction "~{RESET}") (pintype "input"))
     (pad "9" smd rect locked (at -6 -3.7 270) (size 1.8 0.8) (layers "B.Cu" "B.Paste" "B.Mask")
       (net 33 "Net-(R11-Pad1)") (pinfunction "VCC_RF") (pintype "power_out"))
@@
       (net 35 "unconnected-(U3-Pad17)") (pinfunction "RESERVED") (pintype "no_connect"))
     (pad "18" smd rect locked (at 6 0.4 270) (size 1.8 0.8) (layers "B.Cu" "B.Paste" "B.Mask")
-      (net 31 "Net-(R8-Pad1)") (pinfunction "SDA/~SPI_CS") (pintype "bidirectional"))
+      (net 31 "Net-(R8-Pad1)") (pinfunction "SDA/~{SPI_CS}") (pintype "bidirectional"))
     (pad "19" smd rect locked (at 6 1.5 270) (size 1.8 0.8) (layers "B.Cu" "B.Paste" "B.Mask")
       (net 32 "Net-(R9-Pad1)") (pinfunction "SCL/SPI_CLK") (pintype "input"))
@@
     (fp_line (start -1.4 -0.3) (end -1.4 0.3) (layer "B.SilkS") (width 0.12))
     (fp_line (start -0.7 1) (end 0.7 1) (layer "B.SilkS") (width 0.12))
-    (fp_arc (start 0.7 -0.3) (end 0.7 -1) (angle 90) (layer "B.SilkS") (width 0.12))
-    (fp_arc (start 0.7 0.3) (end 1.4 0.3) (angle 90) (layer "B.SilkS") (width 0.12))
-    (fp_arc (start -0.7 0.3) (end -0.7 1) (angle 90) (layer "B.SilkS") (width 0.12))
-    (fp_arc (start -0.7 -0.3) (end -1.4 -0.3) (angle 90) (layer "B.SilkS") (width 0.12))
+    (fp_arc (start 0.7 -1) (mid 1.194975 -0.794975) (end 1.4 -0.3) (layer "B.SilkS") (width 0.12))
+    (fp_arc (start 1.4 0.3) (mid 1.194975 0.794975) (end 0.7 1) (layer "B.SilkS") (width 0.12))
+    (fp_arc (start -0.7 1) (mid -1.194975 0.794975) (end -1.4 0.3) (layer "B.SilkS") (width 0.12))
+    (fp_arc (start -1.4 -0.3) (mid -1.194975 -0.794975) (end -0.7 -1) (layer "B.SilkS") (width 0.12))
     (fp_line (start -1.65 1.25) (end 1.65 1.25) (layer "B.CrtYd") (width 0.05))
     (fp_line (start 1.65 -1.25) (end -1.65 -1.25) (layer "B.CrtYd") (width 0.05))
@@
         (gr_circle (center 0 0.25) (end 0.5 0.25) (width 0) (fill yes))
         (gr_poly (pts
-          (xy 0 0.75)
-          (xy 0.5 0.75)
-          (xy 0.5 -0.75)
-          (xy 0 -0.75)
-        ) (width 0) (fill yes))
+            (xy 0.5 0.75)
+            (xy 0 0.75)
+            (xy 0 -0.75)
+            (xy 0.5 -0.75)
+          ) (width 0) (fill yes))
       ))
     (pad "2" smd custom locked (at 0.65 0 270) (size 1 0.5) (layers "B.Cu" "B.Mask")
@@
         (gr_circle (center 0 0.25) (end 0.5 0.25) (width 0) (fill yes))
         (gr_poly (pts
-          (xy 0 0.75)
-          (xy -0.5 0.75)
-          (xy -0.5 -0.75)
-          (xy 0 -0.75)
-        ) (width 0) (fill yes))
+            (xy 0 0.75)
+            (xy -0.5 0.75)
+            (xy -0.5 -0.75)
+            (xy 0 -0.75)
+          ) (width 0) (fill yes))
       ))
   )
@@
       (effects (font (size 1 1) (thickness 0.15)) (justify mirror))
     )
-    (fp_text value "BC817-25" (at 0 -2.5) (layer "B.Fab")
+    (fp_text value "BC817-25" (at 0 -2.5) (layer "B.Fab") hide
       (effects (font (size 1 1) (thickness 0.15)) (justify mirror))
     )
@@
     (fp_line (start -0.7 -1.52) (end 0.7 -1.52) (layer "B.Fab") (width 0.1))
     (pad "1" smd rect locked (at -1 0.95 180) (size 0.9 0.8) (layers "B.Cu" "B.Paste" "B.Mask")
-      (net 20 "Net-(Q1-Pad1)") (pinfunction "B"))
+      (net 20 "Net-(Q1-Pad1)") (pinfunction "B") (pintype "input"))
     (pad "2" smd rect locked (at -1 -0.95 180) (size 0.9 0.8) (layers "B.Cu" "B.Paste" "B.Mask")
-      (net 1 "GND") (pinfunction "E"))
+      (net 1 "GND") (pinfunction "E") (pintype "passive"))
     (pad "3" smd rect locked (at 1 0 180) (size 0.9 0.8) (layers "B.Cu" "B.Paste" "B.Mask")
-      (net 47 "Net-(Q1-Pad3)") (pinfunction "C"))
+      (net 47 "Net-(Q1-Pad3)") (pinfunction "C") (pintype "passive"))
     (model "${KISYS3DMOD}/Package_TO_SOT_SMD.3dshapes/SOT-23.wrl"
       (offset (xyz 0 0 0))
