File: hw/sch_pcb/GPS02B.kicad_sch (KiCad schematic)
At the start: 63 parts, among them J1 HEADER_2x03_PARALLEL, J10 HEADER_2x01_PARALLEL, J11 HEADER_2x01_PARALLEL, J12 HEADER_2x01_PARALLEL, J13 HEADER_2x01_PARALLEL, J14 HEADER_2x01_PARALLEL, J15 HEADER_2x03_PARALLEL, J16 HEADER_2x01_PARALLEL, J17 u.FL, J18 SMA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

Commit message: Edit #5 #4 #3 #1
Parts:
- removed J17: u.FL, Connector_Coaxial:U.FL_Molex_MCRF_73412-0110_Vertical, symbol GPS02A-rescue:SMA-MLAB_CONNECTORS
- removed R14: 620R, Mlab_R:SMD-0805, symbol GPS02A-rescue:R-Device
- added Q1: BC817-25, Package_TO_SOT_SMD:SOT-23, symbol Device:Q_NPN_BEC
- added R14, R16: 220R, Mlab_R:SMD-0805, symbol Device:R
- C7: value 10nF -> 47pF; UST_ID 5c70984712875079b91f8b49 -> (none)
- D1: value BAS85 -> M4; footprint Diode_SMD:D_MiniMELF -> Diode_SMD:D_SMA
- J18: footprint Connector_Coaxial:SMB_Jack_Vertical -> Mlab_CON:SMA6251A13G50
- L2: footprint Mlab_R:SMD-0805 -> Inductor_SMD:L_0402_1005Metric; UST_ID 5c70984412875079b91f8807 -> (none)
Connections:
- net +3V3: now also D6.2 (A)
- net GND: now also Q1.2 (E)
- net TIMEPULSE: now also R14.1; no longer D6.2 (A)
- net at D6.1 (K): now also R16.2
- new net: Q1.1 (B), R14.2
- new net: Q1.3 (C), R16.1
Other:
- moved on the sheet: C6, D6, J15

Commit message: Edit bom
Parts:
- C7: UST_ID (none) -> 5c70984712875079b91f8b38
- L2: UST_ID (none) -> 618cbf071287506e2801ed7e
Changed lines of the file:
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@@
-(kicad_sch (version 20210406) (generator eeschema)
+(kicad_sch (version 20210621) (generator eeschema)
   (paper "A4")
   (title_block
@@
       (effects (font (size 1.27 1.27)) hide)
     )
-    (property "UST_ID" "" (id 4) (at 175.26 80.01 0)
+    (property "UST_ID" "618cbf071287506e2801ed7e" (id 4) (at 175.26 80.01 0)
       (effects (font (size 1.27 1.27)) hide)
     )
@@
       (effects (font (size 1.27 1.27)) hide)
     )
-    (property "UST_ID" "" (id 4) (at 185.42 80.01 0)
-      (effects (font (size 1.27 1.27)) hide)
-    )
+    (property "UST_ID" "5c70984712875079b91f8b38" (id 4) (at 185.42 80.01 0)
+      (effects (font (size 1.27 1.27)) hide)
+    )

Commit message: Edit BOM
Parts:
- D1: UST_ID 5c70984512875079b91f88b3 -> 5c70984512875079b91f88ac
Changed lines of the file:
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@@
       (effects (font (size 1.27 1.27)) hide)
     )
-    (property "UST_ID" "5c70984512875079b91f88b3" (id 4) (at 19.05 115.57 0)
+    (property "UST_ID" "5c70984512875079b91f88ac" (id 4) (at 19.05 115.57 0)
       (effects (font (size 1.27 1.27)) hide)
     )

Commit message: Update link to datasheet Update titleblock.
Other:
- title: NAME -> GPS02B
